File: BCP/Main.kicad_pcb (KiCad board)
At the start: 2 copper layers, 6 parts, among them SW1 SW_Nidec_CAS-120A1, U1 LD1117V33, U2 Pico 2, U3 DEV-13712, U4 NEO-M9N

Commit message: Added GPS (somewhat)
Parts:
- removed U4: NEO-M9N, Trantor:NEO-M9N
Routing:
- net Net-(SW1-A): track 0.00 -> 20.9 mm
- net Net-(BT2-+): track 0.00 -> 13.8 mm

Commit message: Removed autosave (I swear I know what I'm doing)
Connections:
- U2 pad 24: unconnected-(U2-GPIO18-Pad24) -> /FLIGHTLED
- U2 pad 25: unconnected-(U2-GPIO19-Pad25) -> /DEBUG3
- U2 pad 26: unconnected-(U2-GPIO20-Pad26) -> /DEBUG2
- U2 pad 27: unconnected-(U2-GPIO21-Pad27) -> /DEBUG1
Changed lines of the file:
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@@
 	(net 20 "unconnected-(U2-VBUS-Pad40)")
 	(net 21 "unconnected-(U2-GPIO9-Pad12)")
-	(net 22 "unconnected-(U2-GPIO20-Pad26)")
+	(net 22 "/DEBUG2")
 	(net 23 "unconnected-(U2-SWCLK-Pad41)")
-	(net 24 "unconnected-(U2-GPIO19-Pad25)")
+	(net 24 "/DEBUG3")
 	(net 25 "unconnected-(U2-GND-Pad13)")
 	(net 26 "unconnected-(U2-GPIO26_ADC0-Pad31)")
@@
 	(net 41 "unconnected-(U2-GPIO11-Pad15)")
 	(net 42 "unconnected-(U2-GND-Pad18)")
-	(net 43 "unconnected-(U2-GPIO21-Pad27)")
-	(net 44 "unconnected-(U2-GPIO18-Pad24)")
+	(net 43 "/DEBUG1")
+	(net 44 "/FLIGHTLED")
 	(net 45 "unconnected-(U2-GPIO6-Pad9)")
 	(net 46 "unconnected-(U2-GPIO28_ADC2-Pad34)")
@@
 			(layers "*.Cu" "*.Mask")
 			(remove_unused_layers no)
-			(net 44 "unconnected-(U2-GPIO18-Pad24)")
+			(net 44 "/FLIGHTLED")
 			(pinfunction "GPIO18")
 			(pintype "bidirectional")
@@
 			)
 			(layers "F.Cu" "F.Mask")
-			(net 44 "unconnected-(U2-GPIO18-Pad24)")
+			(net 44 "/FLIGHTLED")
 			(pinfunction "GPIO18")
 			(pintype "bidirectional")
@@
 			(layers "*.Cu" "*.Mask")
 			(remove_unused_layers no)
-			(net 24 "unconnected-(U2-GPIO19-Pad25)")
+			(net 24 "/DEBUG3")
 			(pinfunction "GPIO19")
 			(pintype "bidirectional")
@@
 			)
 			(layers "F.Cu" "F.Mask")
-			(net 24 "unconnected-(U2-GPIO19-Pad25)")
+			(net 24 "/DEBUG3")
 			(pinfunction "GPIO19")
 			(pintype "bidirectional")
@@
 			(layers "*.Cu" "*.Mask")
 			(remove_unused_layers no)
-			(net 22 "unconnected-(U2-GPIO20-Pad26)")
+			(net 22 "/DEBUG2")
 			(pinfunction "GPIO20")
 			(pintype "bidirectional")
@@
 			)
 			(layers "F.Cu" "F.Mask")
-			(net 22 "unconnected-(U2-GPIO20-Pad26)")
+			(net 22 "/DEBUG2")
 			(pinfunction "GPIO20")
 			(pintype "bidirectional")
@@
 			(layers "*.Cu" "*.Mask")
 			(remove_unused_layers no)
-			(net 43 "unconnected-(U2-GPIO21-Pad27)")
+			(net 43 "/DEBUG1")
 			(pinfunction "GPIO21")
 			(pintype "bidirectional")
@@
 			)
 			(layers "F.Cu" "F.Mask")
-			(net 43 "unconnected-(U2-GPIO21-Pad27)")
+			(net 43 "/DEBUG1")
 			(pinfunction "GPIO21")
 			(pintype "bidirectional")

Commit message: Added GPS and BME
Parts:
- added U4: ~, Trantor:GPS, F.Cu at (122.0, 147.4)

Commit message: Theoretically done?
Parts:
- added U5: ~, Trantor:BNO055, F.Cu at (156.8, 67.8)
- added U6: BME280, Trantor:BME280, F.Cu at (94.8, 112.2)
- U3: value DEV-13712 -> Logger
- moved U3 61.7 mm to (161.5, 97.8), turned to 180 degrees
- moved SW1 61.4 mm to (165.7, 48.2), turned to 0 degrees
- moved U1 39.7 mm to (158.2, 46.0), turned to 90 degrees
- moved U4 33.5 mm to (141.2, 120.0)
- moved U2 31.1 mm to (126.4, 56.2)
- moved BT2 20.6 mm to (98.8, 38.8)
Routing:
- net unconnected-(U2-GPIO2-Pad4): track 0.00 -> 20.9 mm
- net Net-(SW1-A): track 20.9 -> 0.00 mm
- net unconnected-(U2-GPIO6-Pad9): track 0.00 -> 13.8 mm
- net Net-(BT2-+): track 13.8 -> 0.00 mm
Other:
- board outline added: 20.3 x 26.7 mm

Commit message: Grouped Like Components
Parts:
- U3: value Logger -> DEV-13712
- moved SW1 99.9 mm to (85.8, 108.2)
- moved U1 99.9 mm to (78.4, 106.0)
- moved U6 88.9 mm to (157.0, 48.8), turned to -90 degrees
- moved U5 3.02 mm to (155.5, 70.5), turned to 180 degrees
Routing:
- net unconnected-(U2-GPIO2-Pad4): track 20.9 -> 0.00 mm
- net unconnected-(U2-GPIO6-Pad9): track 13.8 -> 0.00 mm
Other:
- board outline removed
