File: BCPMainCircuit/BCPMainCircuit.kicad_sch (KiCad schematic)
At the start: 21 parts, among them Q1 IRLB8721PBF, SW1 Switch, U2 Pico 2, U3 Logger, U4 GPS, U5 BNO055, U6 BME280, U7 MIC2940A-3.3WT

Commit message: Major changes: Added 2x 8:1 multiplexers for thermocouples, up to 8, can be selected using pins 19,20,21 IN REVERSE ORDER! Added 1 primary TC amp, with capacity for 2 extra using ADC 0,1,2 Moved flight leds to near pico (prob gonna change that, but im too tired rn
Minor changes:
Flight leds share a resistor now since they use constant current
moved some stuff i think
Debug leds moved to 7,8,9 IN REVERSE ORDER!
other stuff?
Parts:
- removed R2: ???R, Resistor_THT:R_Axial_DIN0207_L6.3mm_D2.5mm_P7.62mm_Horizontal, symbol Device:R_Small_US
- added MU1, MU2: ~, Gabriel_footprints:74HC4051 8_1, symbol My_Stuff:8{colon}1_Mux
- added TC1, TC2, TC3, TC4, TC5, TC6, TC7, TC8: Thermocouple, symbol Device:Thermocouple
- added TCA1, TCA2, TCA3: AD8495 Breakout, Gabriel_footprints:AD8495 Breakout, symbol My_Stuff:AD8495_Breakout
Connections:
- net +3.3V: now also MU1.10 (VCC), MU1.2 (VCC), MU2.10 (VCC), MU2.2 (VCC), TCA1.1 (V+), TCA2.1 (V+), TCA3.1 (V+)
- net DEBUG1: now also U2.12 (GPIO9); no longer U2.27 (GPIO21)
- net DEBUG2: now also U2.11 (GPIO8); no longer U2.26 (GPIO20)
- net DEBUG3: now also U2.10 (GPIO7); no longer U2.25 (GPIO19)
- net GND: now also MU1.11 (GND), MU1.3 (GND), MU2.11 (GND), MU2.3 (GND), TCA1.2 (GND), TCA1.4 (GND), TCA2.2 (GND), TCA2.4 (GND), TCA3.2 (GND), TCA3.4 (GND)
- net ThermoAmp1: now reaches U2.31 (GPIO26_ADC0)
- net ThermoAmp1: now also TCA1.3 (OUT)
- net ThermoAmp2: now reaches U2.32 (GPIO27_ADC1)
- net ThermoAmp2: now also TCA2.3 (OUT)
- net ThermoAmp3: now reaches U2.34 (GPIO28_ADC2)
- net ThermoAmp3: now also TCA3.3 (OUT)
- net at D1.2 (A), R1.2: now also D5.2 (A)
- new net TC+1: MU1.12 (Y0), TC1.1 (+)
- new net TC+2: MU1.13 (Y1), TC2.1 (+)
- new net TC+3: MU1.14 (Y2), TC3.1 (+)
- new net TC+4: MU1.15 (Y3), TC4.1 (+)
- new net TC+5: MU1.16 (Y4), TC5.1 (+)
- new net TC+6: MU1.17 (Y5), TC6.1 (+)
- new net TC+7: MU1.18 (Y6), TC7.1 (+)
- new net TC+8: MU1.19 (Y7), TC8.1 (+)
- new net TC+YLW: MU1.4 (Z), TCA1.5 (YLW+)
- new net TC-1: MU2.12 (Y0), TC1.2 (-)
- new net TC-2: MU2.13 (Y1), TC2.2 (-)
- new net TC-3: MU2.14 (Y2), TC3.2 (-)
- new net TC-4: MU2.15 (Y3), TC4.2 (-)
- new net TC-5: MU2.16 (Y4), TC5.2 (-)
- new net TC-6: MU2.17 (Y5), TC6.2 (-)
- new net TC-7: MU2.18 (Y6), TC7.2 (-)
- new net TC-8: MU2.19 (Y7), TC8.2 (-)
- new net TC-RED: MU2.4 (Z), TCA1.6 (RED-)
- new net TC-Sel1: MU1.5 (S0), MU2.5 (S0), U2.27 (GPIO21)
- new net TC-Sel2: MU1.6 (S1), MU2.6 (S1), U2.26 (GPIO20)
- new net TC-Sel3: MU1.7 (S2), MU2.7 (S2), U2.25 (GPIO19)
- no-connect marks 24 -> 30
Other:
- note added: "NOTES Flight LED moved to GPIO22 Debug LEDs moved to GPIO 7,8,9 IN REVERSE ORDER! ThermoSelect pins are 19,20,21 IN REVERSE ORDER! note: to use, just set the pins you need high, i can explain later"
- note added: "Thermals"
- note added: "note to self: make SURE the + and - of each TC are connected to the CORRECT PINS because IT MATTERS"
- note removed: "NOTES Flight LED moved to GPIO22"
- moved on the sheet: C1, C2, Q1, R1, R3, R4, R5, U7

Commit message: Major changes: Removed TC amps, replaced with SMD TC amps instead idk
Parts:
- removed TCA1, TCA2, TCA3: AD8495 Breakout, Gabriel_footprints:AD8495 Breakout, symbol My_Stuff:AD8495_Breakout
- added C3, C4: 0u1f, Capacitor_SMD:C_0201_0603Metric, symbol Device:C_Small
- added R10, R11, R13, R14: 100, Resistor_SMD:R_0201_0603Metric, symbol Device:R_US
- added R12, R16, R6, R7: 2M, Resistor_SMD:R_0201_0603Metric, symbol Device:R_US
- added R15, R5: 1M, Resistor_SMD:R_0201_0603Metric, symbol Device:R_US
- added R17, R18, R8, R9: 10k, Resistor_SMD:R_0201_0603Metric, symbol Device:R_US
- added U1, U8: MCP9601T-E/MX, MQFN20_NU_MCH, symbol SMD_TC_AMP:MCP9601T-E_MX
- TC2: footprint (none) -> Connector_PinHeader_2.54mm:PinHeader_1x02_P2.54mm_Vertical
- renumbered R3 to R2, R4 to R3, R5 to R4
Connections:
- net +3.3V: now also R15.2, R17.1, R18.1, R5.2, R8.1, R9.1, U1.8 (VDD), U8.8 (VDD)
- net GND: now also R12.2, R16.1, R6.1, R7.2, U1.1 (GND), U1.10 (GND), U1.13 (GND), U1.16 (ADDR), U1.17 (GND), U1.18 (GND), U1.21 (GND), U1.3 (GND), U1.5 (GND), U8.1 (GND), U8.10 (GND), U8.13 (GND), U8.16 (ADDR), U8.17 (GND), U8.18 (GND), U8.21 (GND), U8.3 (GND), U8.5 (GND)
- net SCL: now also R18.2, R8.2, U1.19 (SCL), U8.19 (SCL)
- net SDA: now also R17.2, R9.2, U1.20 (SDA), U8.20 (SDA)
- net TC+2: now also R14.1
- net TC+YLW: now also R10.1
- net TC-2: now also R12.1, R13.1
- net TC-RED: now also R11.1, R7.1
- net ThermoSCwarn: now reaches U2.21 (GPIO16)
- net ThermoSCwarn: now also U1.7 (SCALERT), U8.7 (SCALERT)
- net ThermoOCwarn: now reaches U2.22 (GPIO17)
- net ThermoOCwarn: now also U1.9 (OCALERT), U8.9 (OCALERT)
- net ThermoAmp1: no longer names the net of U2.31 (GPIO26_ADC0)
- net ThermoAmp2: no longer names the net of U2.32 (GPIO27_ADC1)
- net ThermoAmp3: no longer names the net of U2.34 (GPIO28_ADC2)
- new net: C3.1, R10.2, U1.2 (VIN+)
- new net: C3.2, R11.2, U1.4 (VIN-)
- new net: C4.1, R14.2, U8.2 (VIN+)
- new net: C4.2, R13.2, U8.4 (VIN-)
- new net VSense1: R5.1, R6.2, U1.6 (VSENSE)
- new net VSense2: R15.1, R16.2, U8.6 (VSENSE)
Other:
- note added: "60"
- note added: "61"
- note added: "62"
- note added: "63"
- note added: "64"
- note added: "65"
- note added: "66"
- note added: "67"
- note added: "ADDR: 29/28"
- note added: "ADDR: 42"
- note added: "ADDR: 76/77"
- moved on the sheet: C1, C2, Q1, R1, R2, R3, R4, U7
