File: BCPMainCircuit/BCPMainCircuit.kicad_sch (KiCad schematic)
At the start: 64 parts, among them J1 MSD-4-A, Q1 IRLB8721PBF, SW1 Switch, U1 MCP9601T-E/MX, U10 LSM6DSO, U2 Pico 2, U3 NEO-M9N-00B, U5 BME280, U6 CD4097B, U7 LIS2MDL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

Commit message: Replaced mux with different, smaller, smd, cheaper one put flight leds back
NEED TO DO:
add gps antenna
check if gps needs filter caps
verify v. reg capacitors (size, footprint, values)
figure out how sd cards work (im confused by them, for i have a simple mind)
breakout pins for everything we'd want
Parts:
- removed MU1, MU2: ~, Gabriel_footprints:74HC4051 8_1, symbol My_Stuff:8{colon}1_Mux
- U6: footprint (none) -> Package_SO:SOIC-24W_7.5x15.4mm_P1.27mm
Connections:
- net FLIGHTLED: now also U2.14 (GPIO10); no longer U2.29 (GPIO22)
- net TC+1: now also U6.9 (X0)
- net TC+2: now also U6.8 (X1)
- net TC+3: now also U6.7 (X2)
- net TC+4: now also U6.6 (X3)
- net TC+5: now also U6.5 (X4)
- net TC+6: now also U6.4 (X5)
- net TC+7: now also U6.3 (X6)
- net TC+8: now also U6.2 (X7)
- net TC-1: now also U6.23 (Y0)
- net TC-2: now also U6.22 (Y1)
- net TC-3: now also U6.21 (Y2)
- net TC-4: now also U6.20 (Y3)
- net TC-5: now also U6.19 (Y4)
- net TC-6: now also U6.18 (Y5)
- net TC-7: now also U6.16 (Y6)
- net TC-8: now also U6.15 (Y7)
- no-connect marks 30 -> 24
Other:
- note added: "Thermocouples + Multiplexer"
- note removed: "Thermocouples + Multiplexers"
- moved on the sheet: C12, C13, R19, R20, U10, U6

Commit message: added gps antenna sd card is hopefully correct breakout pins added ran drc, only mad about the 0603 sized stuff having insufficient clearance, probably fine
still need someone to verify:
v. reg capacitors n stuff
gps filter caps???
every smd thing lol, its SO BAD
and
software needs to review available breakout pins, as well as other misc. stuff to be sure its good
Parts:
- added AE1: Antenna, Connector_Coaxial:U.FL_Hirose_U.FL-R-SMT-1_Vertical, symbol Device:Antenna
Connections:
- net +3.3V: now also U3.22 (V_BCKP)
- net GND: now also U3.7 (V_USB)
- net at U3.11 (RF_IN): now also AE1.1 (A)
- no-connect marks 24 -> 23
Other:
- moved on the sheet: C10, C11, C12, C13, C14, C15, C2, C4, C6, C7, C8, C9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

Commit message: fixed stuff
Parts:
- C1: value 200nf -> 220nf; footprint Capacitor_SMD:C_0201_0603Metric -> Capacitor_SMD:C_0603_1608Metric
- C12, C13, C14, C15, C2, C3, C4: footprint Capacitor_SMD:C_0201_0603Metric -> Capacitor_SMD:C_0603_1608Metric
- R10, R11, R12, R13, R14, R19, R20, R5, R6, R7, R8, R9: footprint Resistor_SMD:R_0201_0603Metric -> Resistor_SMD:R_0603_1608Metric

Commit message: changed imu
Parts:
- removed C12, C13: 0u1f, Capacitor_SMD:C_0603_1608Metric, symbol Device:C_Small
- removed C14, C15: 100nf, Capacitor_SMD:C_0603_1608Metric, symbol Device:C_Small
- removed C2: 220nf, Capacitor_SMD:C_0603_1608Metric, symbol Device:C_Small
- removed C4: 10uf, Capacitor_SMD:C_0603_1608Metric, symbol Device:C_Small
- removed D6, D7, D8: WS2812, LED_SMD:LED_WS2812_PLCC6_5.0x5.0mm_P1.6mm, symbol LED:WS2812
- removed R14, R19, R20: 10kΩ, Resistor_SMD:R_0603_1608Metric, symbol Device:R_Small_US
- removed U10: LSM6DSO, Gabriel_footprints:LSM6DSO, symbol LSM6DSO:LSM6DSO
- removed U7: LIS2MDL, Package_LGA:LGA-12_2x2mm_P0.5mm, symbol Sensor_Magnetic:LIS2MDL
- added C16: 100nf, Capacitor_SMD:C_0603_1608Metric, symbol Device:C_Small
- added C17, C18: 0u1f, Capacitor_SMD:C_0603_1608Metric, symbol Device:C_Small
- added R15: 10kΩ, Resistor_SMD:R_0603_1608Metric, symbol Device:R_Small_US
- added R18, R21: 4kΩ, Resistor_SMD:R_0603_1608Metric, symbol Device:R_Small_US
- added U4: BNO085, Gabriel_footprints:IC_BNO085, symbol BNO085:BNO085
Connections:
- net +3.3V: now also C17.1, C18.1, R15.1, R18.2, R21.2, U4.10 (CLKSEL0), U4.28 (VDDIO), U4.3 (VDD), U4.5 (PS1)
- net GND: now also U2.28 (GND), C16.2, C17.2, C18.2, U4.2 (GND), U4.25 (GNDIO), U4.26 (XOUT32/CLKSEL1)
- net SD_CS: now also U4.18 (~{H_CS})
- net SD_MISO: now also U4.20 (H_SDA/H_MISO/TX)
- net SD_MOSI: now also U4.17 (SA0/H_MOSI)
- net SD_SCK: now also U4.19 (H_SCL/SCK/RX)
- net IMU_Int: now reaches U2.26 (GPIO20)
- net IMU_Int: now also U4.14 (~{H_INT})
- net IMU_RST: now reaches U2.29 (GPIO22)
- net IMU_RST: now also U4.11 (~{RST})
- net IMU_Wake: now reaches U2.31 (GPIO26_ADC0)
- net IMU_Wake: now also U4.6 (PS0/WAKE)
- new net: C16.1, U4.9 (CAP)
- new net: R21.1, U4.15 (ENV_SCL)
- new net: U4.1 (RESV_NC), U4.12 (RESV_NC), U4.13 (RESV_NC), U4.21 (RESV_NC), U4.22 (RESV_NC), U4.23 (RESV_NC), U4.24 (RESV_NC), U4.7 (RESV_NC), U4.8 (RESV_NC)
- new net: R18.1, U4.16 (ENV_SDA)
- new net IMU_Boot: R15.2, U4.4 (~{BOOT})
- no-connect marks 23 -> 18
Other:
- note removed: "https://learn.adafruit.com/adafruit-dotstar-leds?view=all#power-and-connections"
- note removed: "https://www.adafruit.com/product/2343#technical-details"
- note removed: "these need 5v, need to figure something else out"

Commit message: e
Connections:
- net GND: now also BT2.N1 (-); no longer BT2.2 (-)
- net SD_CS: no longer U4.18 (~{H_CS})
- net IMU_CS: now reaches U2.32 (GPIO27_ADC1)
- net IMU_CS: now also U4.18 (~{H_CS})
- net at SW1.2 (B): now also BT2.P2 (+); no longer BT2.1 (+)
Changed lines of the file:
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@@
 	(wire
 		(pts
-			(xy 149.86 111.76) (xy 146.05 111.76)
+			(xy 149.86 113.03) (xy 148.59 113.03)
 		)
 		(stroke
@@
 	(wire
 		(pts
+			(xy 148.59 113.03) (xy 148.59 111.76)
+		)
+		(stroke
+			(width 0)
+			(type default)
+		)
+	)
+	(wire
+		(pts
 			(xy 321.31 91.44) (xy 318.77 91.44)
 		)
@@
 	(wire
 		(pts
+			(xy 148.59 109.22) (xy 146.05 109.22)
+		)
+		(stroke
+			(width 0)
+			(type default)
+		)
+	)
+	(wire
+		(pts
 			(xy 44.45 237.49) (xy 44.45 250.19)
 		)
@@
 	(wire
 		(pts
+			(xy 148.59 111.76) (xy 146.05 111.76)
+		)
+		(stroke
+			(width 0)
+			(type default)
+		)
+	)
+	(wire
+		(pts
 			(xy 238.76 74.93) (xy 236.22 74.93)
 		)
@@
 	)
 	(label "IMU_Wake"
-		(at 149.86 111.76 0)
+		(at 149.86 113.03 0)
 		(effects
 			(font
@@
 		)
 	)
-	(global_label "SD_CS"
+	(global_label "IMU_CS"
 		(shape input)
 		(at 295.91 207.01 180)
@@
 		)
 		(property "Intersheetrefs" "${INTERSHEET_REFS}"
-			(at 286.9982 207.01 0)
+			(at 286.091 207.01 0)
 			(effects
 				(font
@@
 		)
 	)
+	(global_label "IMU_CS"
+		(shape input)
+		(at 148.59 109.22 0)
+		(fields_autoplaced yes)
+		(effects
+			(font
+				(size 1.27 1.27)
+			)
+			(justify left)
+		)
+		(property "Intersheetrefs" "${INTERSHEET_REFS}"
+			(at 158.409 109.22 0)
+			(effects
+				(font
+					(size 1.27 1.27)
+				)
+				(justify left)
+				(hide yes)
+			)
+		)
+	)
 	(global_label "SD_MISO"
 		(shape input)
@@
 			)
 		)
-		(pin "2"
+		(pin "P2"
 		)
-		(pin "1"
+		(pin "N1"
 		)
 		(instances

Commit message: e
Parts:
- C16: value 100nf -> 0u1f
- C7: value 100nF -> 0u1F
Changed lines of the file:
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@@
 	(rectangle
 		(start 15.24 17.78)
-		(end 87.63 206.375)
+		(end 87.63 125.095)
 		(stroke
 			(width 0)
@@
 			)
 		)
-		(property "Value" "100nF"
+		(property "Value" "0u1F"
 			(at 90.932 249.936 0)
 			(effects
@@
 			)
 		)
-		(property "Value" "100nf"
+		(property "Value" "0u1f"
 			(at 371.094 209.296 0)
 			(effects

Commit message: changed the battery holder size, hope it's not too close to the edge
Parts:
- removed BT2: Batteries, Gabriel_footprints:BAT_1079, symbol Device:Battery
- added BT1: 1097P, Gabriel_footprints:BAT_1097P, symbol 1097P:1097P
Connections:
- net GND: now also BT1.N2
- net at SW1.2 (B): now also BT1.P1
- new net: BT1.N1, BT1.P2
Changed lines of the file:
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@@
 	(wire
 		(pts
-			(xy 21.59 231.14) (xy 22.86 231.14)
-		)
-		(stroke
-			(width 0)
-			(type default)
-		)
-	)
-	(wire
-		(pts
 			(xy 187.96 194.31) (xy 194.31 194.31)
 		)
@@
 	(wire
 		(pts
-			(xy 21.59 236.22) (xy 21.59 231.14)
-		)
-		(stroke
-			(width 0)
-			(type default)
-		)
-	)
-	(wire
-		(pts
 			(xy 294.64 49.53) (xy 294.64 52.07)
 		)
@@
 	(wire
 		(pts
+			(xy 19.05 231.14) (xy 19.05 238.76)
+		)
+		(stroke
+			(width 0)
+			(type default)
+		)
+	)
+	(wire
+		(pts
 			(xy 115.57 29.21) (xy 119.38 29.21)
 		)
@@
 	(wire
 		(pts
+			(xy 34.29 241.3) (xy 34.29 238.76)
+		)
+		(stroke
+			(width 0)
+			(type default)
+		)
+	)
+	(wire
+		(pts
 			(xy 377.19 200.66) (xy 387.35 200.66)
 		)
@@
 	(wire
 		(pts
-			(xy 33.02 231.14) (xy 34.29 231.14)
-		)
-		(stroke
-			(width 0)
-			(type default)
-		)
-	)
-	(wire
-		(pts
 			(xy 149.86 129.54) (xy 146.05 129.54)
 		)
@@
 	)
 	(symbol
+		(lib_id "1097P:1097P")
+		(at 26.67 236.22 0)
+		(mirror y)
+		(unit 1)
+		(exclude_from_sim no)
+		(in_bom yes)
+		(on_board yes)
+		(dnp no)
+		(property "Reference" "BT1"
+			(at 26.67 223.52 0)
+			(effects
+				(font
+					(size 1.27 1.27)
+				)
+			)
+		)
+		(property "Value" "1097P"
+			(at 26.67 226.06 0)
+			(effects
+				(font
+					(size 1.27 1.27)
+				)
+			)
+		)
+		(property "Footprint" "Gabriel_footprints:BAT_1097P"
+			(at 26.67 236.22 0)
+			(effects
+				(font
+					(size 1.27 1.27)
+				)
+				(justify bottom)
+				(hide yes)
+			)
+		)
+		(property "Datasheet" ""
+			(at 26.67 236.22 0)
+			(effects
+				(font
+					(size 1.27 1.27)
+				)
+				(hide yes)
+			)
+		)
+		(property "Description" ""
+			(at 26.67 236.22 0)
+			(effects
+				(font
+					(size 1.27 1.27)
+				)
+				(hide yes)
+			)
+		)
+		(property "PARTREV" "A"
+			(at 26.67 236.22 0)
+			(effects
+				(font
+					(size 1.27 1.27)
+				)
+				(justify bottom)
+				(hide yes)
+			)
+		)
+		(property "STANDARD" "Manufacturer Recommendations"
+			(at 26.67 236.22 0)
+			(effects
+				(font
+					(size 1.27 1.27)
+				)
+				(justify bottom)
+				(hide yes)
+			)
+		)
+		(property "SNAPEDA_PN" "1097P"
+			(at 26.67 236.22 0)
+			(effects
+				(font
+					(size 1.27 1.27)
+				)
+				(justify bottom)
+				(hide yes)
+			)
+		)
+		(property "MAXIMUM_PACKAGE_HEIGHT" "15.11mm"
+			(at 26.67 236.22 0)
+			(effects
+				(font
+					(size 1.27 1.27)
+				)
+				(justify bottom)
+				(hide yes)
+			)
+		)
+		(property "MANUFACTURER" "Keystone"
+			(at 26.67 236.22 0)
+			(effects
+				(font
+					(size 1.27 1.27)
+				)
+				(justify bottom)
+				(hide yes)
+			)
+		)
+		(pin "N1"
+		)
+		(pin "P1"
+		)
+		(pin "N2"
+		)
+		(pin "P2"
+		)
+		(instances
+			(project ""
+				(path "/265d59aa-caac-4c2d-9db5-2e2b992cffbc"
+					(reference "BT1")
+					(unit 1)
+				)
+			)
+		)
+	)
+	(symbol
 		(lib_id "power:GND")
 		(at 128.27 57.15 0)
@@
 	(symbol
 		(lib_id "power:GND")
-		(at 21.59 236.22 0)
+		(at 34.29 241.3 0)
 		(unit 1)
 		(exclude_from_sim no)
@@
 		(fields_autoplaced yes)
 		(property "Reference" "#PWR01"
-			(at 21.59 242.57 0)
+			(at 34.29 247.65 0)
 			(effects
 				(font
@@
 		)
 		(property "Value" "GND"
-			(at 21.59 241.3 0)
+			(at 34.29 246.38 0)
 			(effects
 				(font
@@
 		)
 		(property "Footprint" ""
-			(at 21.59 236.22 0)
+			(at 34.29 241.3 0)
 			(effects
 				(font
@@
 		)
 		(property "Datasheet" ""
-			(at 21.59 236.22 0)
+			(at 34.29 241.3 0)
 			(effects
 				(font
@@
 		)
 		(property "Description" "Power symbol creates a global label with name \"GND\" , ground"
-			(at 21.59 236.22 0)
+			(at 34.29 241.3 0)
 			(effects
 				(font
@@
 					(unit 1)
 				)
-			)
-		)
-	)
-	(symbol
-		(lib_id "Device:Battery")
-		(at 27.94 231.14 270)
-		(unit 1)
-		(exclude_from_sim no)
-		(in_bom yes)
-		(on_board yes)
-		(dnp no)
-		(property "Reference" "BT2"
-			(at 28.5115 223.52 90)
-			(effects
-				(font
-					(size 1.27 1.27)
-				)
-				(hide yes)
-			)
-		)
-		(property "Value" "Batteries"
-			(at 27.94 227.33 90)
-			(effects
-				(font
-					(size 1.27 1.27)
-				)
-			)
-		)
-		(property "Footprint" "Gabriel_footprints:BAT_1079"
-			(at 29.464 231.14 90)
-			(effects
-				(font
-					(size 1.27 1.27)
-				)
-				(hide yes)
-			)
-		)
-		(property "Datasheet" "~"
-			(at 29.464 231.14 90)
-			(effects
-				(font
-					(size 1.27 1.27)
-				)
-				(hide yes)
-			)
-		)
-		(property "Description" "Multiple-cell battery"
-			(at 27.94 231.14 0)
-			(effects
-				(font
-					(size 1.27 1.27)
-				)
-				(hide yes)
-			)
-		)
-		(property "Availability" ""
-			(at 27.94 231.14 90)
-			(effects
-				(font
-					(size 1.27 1.27)
-				)
-				(hide yes)
-			)
-		)
-		(property "Check_prices" ""
-			(at 27.94 231.14 90)
-			(effects
-				(font
-					(size 1.27 1.27)
-				)
-				(hide yes)
-			)
-		)
-		(property "Description_1" ""
-			(at 27.94 231.14 90)
-			(effects
-				(font
-					(size 1.27 1.27)
-				)
-				(hide yes)
-			)
-		)
-		(property "MF" ""
-			(at 27.94 231.14 90)
-			(effects
-				(font
-					(size 1.27 1.27)
-				)
-				(hide yes)
-			)
-		)
-		(property "MP" ""
-			(at 27.94 231.14 90)
-			(effects
-				(font
-					(size 1.27 1.27)
-				)
-				(hide yes)
-			)
-		)
-		(property "Package" ""
-			(at 27.94 231.14 90)
-			(effects
-				(font
-					(size 1.27 1.27)
-				)
-				(hide yes)
-			)
-		)
-		(property "Price" ""
-			(at 27.94 231.14 90)
-			(effects
-				(font
-					(size 1.27 1.27)
-				)
-				(hide yes)
-			)
-		)
-		(property "SNAPEDA_PN" ""
-			(at 27.94 231.14 90)
-			(effects
-				(font
-					(size 1.27 1.27)
-				)
-				(hide yes)
-			)
-		)
-		(property "SnapEDA_Link" ""
-			(at 27.94 231.14 90)
-			(effects
-				(font
-					(size 1.27 1.27)
-				)
-				(hide yes)
-			)
-		)
-		(pin "P2"
-		)
-		(pin "N1"
-		)
-		(instances
-			(project ""
-				(path "/265d59aa-caac-4c2d-9db5-2e2b992cffbc"
-					(reference "BT2")
-					(unit 1)
-				)

Commit message: cleanup
Parts:
- removed AE1: Antenna, Connector_Coaxial:U.FL_Hirose_U.FL-R-SMT-1_Vertical, symbol Device:Antenna
- added AE1: Antenna_Shield, Connector_Coaxial:U.FL_Hirose_U.FL-R-SMT-1_Vertical, symbol Device:Antenna_Shield
Connections:
- net GND: now also AE1.2 (Shield)
- net at U3.11 (RF_IN): now also AE1.1 (A)
- no-connect marks 18 -> 22
Other:
- note added: "Atmospheric Sensor"
- note added: "GPS"
- note added: "SD Card Slot"
- note removed: "Check Capacitor/Resistor sizes!!!!!!!!"
- note removed: "SMD components make the jst connector 1x4 instead of 2 1x2s Breakout pins consider 16:2 SMD Mux"
- note removed: "Sensors"
- note removed: "gps antenna?????? Backup battery for faster start??? btw timepulse is a good error indicator capacitors????"
- note removed: "https://www.sparkfun.com/sparkfun-multiplexer-breakout-8-channel-74hc4051.html"
- note removed: "note to self: make SURE the + and - of each TC are connected to the CORRECT PINS because IT MATTERS"
- note removed: "sd cd = card detect"
- note removed: "wtf is happening??"
- moved on the sheet: BT1, C1, C10, C11, C16, C17, C18, C3, C5, C6, C7, C8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
