File: SATURN/OBC/MCU_Power.kicad_sch (KiCad schematic)
At the start: 18 parts

Commit message: usb
Parts:
- renumbered C15 to C10, C16 to C11, C19 to C12, C20 to C13, C21 to C14, C2 to C17, C7 to C2, C5 to C21, C6 to C22, C3 to C25, C4 to C26, C8 to C3, C9 to C4, C10 to C5, C11 to C6, C12 to C7, C13 to C8, C14 to C9
Changed lines of the file:
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@@
 		(on_board yes)
 		(dnp no)
-		(property "Reference" "C14"
+		(property "Reference" "C9"
 			(at 208.28 50.8 90)
 			(effects
@@
 		(on_board yes)
 		(dnp no)
-		(property "Reference" "C13"
+		(property "Reference" "C8"
 			(at 204.47 50.8 90)
 			(effects
@@
 		(on_board yes)
 		(dnp no)
-		(property "Reference" "C20"
+		(property "Reference" "C13"
 			(at 223.52 50.8 90)
 			(effects
@@
 		(dnp no)
 		(fields_autoplaced yes)
-		(property "Reference" "#PWR03"
+		(property "Reference" "#PWR07"
 			(at 153.67 81.28 0)
 			(effects
@@
 		(on_board yes)
 		(dnp no)
-		(property "Reference" "C9"
+		(property "Reference" "C4"
 			(at 189.23 50.8 90)
 			(effects
@@
 		(on_board yes)
 		(dnp no)
-		(property "Reference" "C12"
+		(property "Reference" "C7"
 			(at 200.66 50.8 90)
 			(effects
@@
 		(on_board yes)
 		(dnp no)
-		(property "Reference" "C15"
+		(property "Reference" "C10"
 			(at 212.09 50.8 90)
 			(effects
@@
 		(on_board yes)
 		(dnp no)
-		(property "Reference" "C3"
+		(property "Reference" "C25"
 			(at 162.306 80.01 90)
 			(effects
@@
 		(on_board yes)
 		(dnp no)
-		(property "Reference" "C6"
+		(property "Reference" "C22"
 			(at 162.306 91.44 90)
 			(effects
@@
 		(on_board yes)
 		(dnp no)
-		(property "Reference" "C5"
+		(property "Reference" "C21"
 			(at 162.56 87.63 90)
 			(effects
@@
 		(on_board yes)
 		(dnp no)
-		(property "Reference" "C16"
+		(property "Reference" "C11"
 			(at 215.9 50.8 90)
 			(effects
@@
 		(on_board yes)
 		(dnp no)
-		(property "Reference" "C10"
+		(property "Reference" "C5"
 			(at 193.04 50.8 90)
 			(effects
@@
 		(on_board yes)
 		(dnp no)
-		(property "Reference" "C2"
+		(property "Reference" "C17"
 			(at 112.522 96.774 0)
 			(effects
@@
 		(on_board yes)
 		(dnp no)
-		(property "Reference" "C11"
+		(property "Reference" "C6"
 			(at 196.85 50.8 90)
 			(effects
@@
 		(on_board yes)
 		(dnp no)
-		(property "Reference" "C7"
+		(property "Reference" "C2"
 			(at 181.61 50.8 90)
 			(effects
@@
 		(on_board yes)
 		(dnp no)
-		(property "Reference" "C19"
+		(property "Reference" "C12"
 			(at 219.71 50.8 90)
 			(effects
@@
 		(on_board yes)
 		(dnp no)
-		(property "Reference" "C21"
+		(property "Reference" "C14"
 			(at 227.33 50.8 90)
 			(effects
@@
 		(dnp no)
 		(fields_autoplaced yes)
-		(property "Reference" "#PWR07"
+		(property "Reference" "#PWR0101"
 			(at 237.49 38.1 0)
 			(effects
@@
 		(dnp no)
 		(fields_autoplaced yes)
-		(property "Reference" "#PWR01"
+		(property "Reference" "#PWR02"
 			(at 116.84 105.41 0)
 			(effects
@@
 		(dnp no)
 		(fields_autoplaced yes)
-		(property "Reference" "#PWR06"
+		(property "Reference" "#PWR01"
 			(at 181.61 43.18 0)
 			(effects
@@
 		(on_board yes)
 		(dnp no)
-		(property "Reference" "C8"
+		(property "Reference" "C3"
 			(at 185.42 50.8 90)
 			(effects
@@
 		(dnp no)
 		(fields_autoplaced yes)
-		(property "Reference" "#PWR02"
+		(property "Reference" "#PWR06"
 			(at 152.4 100.33 0)
 			(effects
@@
 		(on_board yes)
 		(dnp no)
-		(property "Reference" "C4"
+		(property "Reference" "C26"
 			(at 162.306 83.82 90)
 			(effects
