File: SATURN/OBC/MCU_Power.kicad_sch (KiCad schematic)
At the start: 18 parts

Commit message: updating stuff
Parts:
- added C1: 220pf, Capacitor_SMD:C_0603_1608Metric, symbol Device:C_Small
- added C17, C18: 10uf, Capacitor_SMD:C_0603_1608Metric, symbol Device:C_Small
- added L1, L2: 2.2uH, symbol Device:L
Connections:
- net GND: now also C1.1, C17.1, C18.1
- new net MCU_VFBSMPS: C17.2, C18.2, L1.2, L2.2
- new net MCU_VLXSMPS: C1.2, L1.1, L2.1
Other:
- moved on the sheet: C2
