File: SATURN/OBC/MCU_Power.kicad_sch (KiCad schematic)
At the start: 18 parts

Commit message: Wired Up Watchdogs. Hopefully correctly.
Parts:
- renumbered C5 to C10, C6 to C11, C7 to C12, C8 to C13, C9 to C14, C10 to C15, C11 to C16, C12 to C19, C17 to C2, C13 to C20, C14 to C21, C25 to C3, C26 to C4, C21 to C5, C22 to C6, C2 to C7, C3 to C8, C4 to C9

Commit message: Added USB switcher and updated to MCUs
Parts:
- renumbered C9 to C10, C10 to C11, C11 to C12, C12 to C13, C13 to C14, C14 to C15, C15 to C16, C16 to C17, C19 to C18, C20 to C19, C21 to C20, C2 to C3, C3 to C4, C4 to C5, C5 to C6, C6 to C7, C7 to C8, C8 to C9
Changed lines of the file:
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@@
 		(in_pos_files yes)
 		(dnp no)
-		(property "Reference" "C14"
+		(property "Reference" "C15"
 			(at 208.28 50.8 90)
 			(show_name no)
@@
 			(project "OBC"
 				(path "/100d4475-6c5b-4ca4-82f4-ff20798e9edf/dc03155b-7cbf-4ee4-9f4c-dba3ed8dc3dd/e4d2ab53-3ce3-4165-a625-695d4175e2ed"
-					(reference "C14")
+					(reference "C15")
 					(unit 1)
 				)
@@
 		(in_pos_files yes)
 		(dnp no)
-		(property "Reference" "C13"
+		(property "Reference" "C14"
 			(at 204.47 50.8 90)
 			(show_name no)
@@
 			(project "OBC"
 				(path "/100d4475-6c5b-4ca4-82f4-ff20798e9edf/dc03155b-7cbf-4ee4-9f4c-dba3ed8dc3dd/e4d2ab53-3ce3-4165-a625-695d4175e2ed"
-					(reference "C13")
+					(reference "C14")
 					(unit 1)
 				)
@@
 		(in_pos_files yes)
 		(dnp no)
-		(property "Reference" "C20"
+		(property "Reference" "C19"
 			(at 223.52 50.8 90)
 			(show_name no)
@@
 			(project "OBC"
 				(path "/100d4475-6c5b-4ca4-82f4-ff20798e9edf/dc03155b-7cbf-4ee4-9f4c-dba3ed8dc3dd/e4d2ab53-3ce3-4165-a625-695d4175e2ed"
-					(reference "C20")
+					(reference "C19")
 					(unit 1)
 				)
@@
 		(dnp no)
 		(fields_autoplaced yes)
-		(property "Reference" "#PWR03"
+		(property "Reference" "#PWR020"
 			(at 153.67 81.28 0)
 			(hide yes)
@@
 			(project "OBC"
 				(path "/100d4475-6c5b-4ca4-82f4-ff20798e9edf/dc03155b-7cbf-4ee4-9f4c-dba3ed8dc3dd/e4d2ab53-3ce3-4165-a625-695d4175e2ed"
-					(reference "#PWR03")
+					(reference "#PWR020")
 					(unit 1)
 				)
@@
 		(in_pos_files yes)
 		(dnp no)
-		(property "Reference" "C9"
+		(property "Reference" "C10"
 			(at 189.23 50.8 90)
 			(show_name no)
@@
 			(project "OBC"
 				(path "/100d4475-6c5b-4ca4-82f4-ff20798e9edf/dc03155b-7cbf-4ee4-9f4c-dba3ed8dc3dd/e4d2ab53-3ce3-4165-a625-695d4175e2ed"
-					(reference "C9")
+					(reference "C10")
 					(unit 1)
 				)
@@
 		(in_pos_files yes)
 		(dnp no)
-		(property "Reference" "C12"
+		(property "Reference" "C13"
 			(at 200.66 50.8 90)
 			(show_name no)
@@
 			(project "OBC"
 				(path "/100d4475-6c5b-4ca4-82f4-ff20798e9edf/dc03155b-7cbf-4ee4-9f4c-dba3ed8dc3dd/e4d2ab53-3ce3-4165-a625-695d4175e2ed"
-					(reference "C12")
+					(reference "C13")
 					(unit 1)
 				)
@@
 		(in_pos_files yes)
 		(dnp no)
-		(property "Reference" "C15"
+		(property "Reference" "C16"
 			(at 212.09 50.8 90)
 			(show_name no)
@@
 			(project "OBC"
 				(path "/100d4475-6c5b-4ca4-82f4-ff20798e9edf/dc03155b-7cbf-4ee4-9f4c-dba3ed8dc3dd/e4d2ab53-3ce3-4165-a625-695d4175e2ed"
-					(reference "C15")
+					(reference "C16")
 					(unit 1)
 				)
@@
 		(in_pos_files yes)
 		(dnp no)
-		(property "Reference" "C3"
+		(property "Reference" "C4"
 			(at 162.306 80.01 90)
 			(show_name no)
@@
 			(project "OBC"
 				(path "/100d4475-6c5b-4ca4-82f4-ff20798e9edf/dc03155b-7cbf-4ee4-9f4c-dba3ed8dc3dd/e4d2ab53-3ce3-4165-a625-695d4175e2ed"
-					(reference "C3")
+					(reference "C4")
 					(unit 1)
 				)
@@
 		(in_pos_files yes)
 		(dnp no)
-		(property "Reference" "C6"
+		(property "Reference" "C7"
 			(at 162.306 91.44 90)
 			(show_name no)
@@
 			(project "OBC"
 				(path "/100d4475-6c5b-4ca4-82f4-ff20798e9edf/dc03155b-7cbf-4ee4-9f4c-dba3ed8dc3dd/e4d2ab53-3ce3-4165-a625-695d4175e2ed"
-					(reference "C6")
+					(reference "C7")
 					(unit 1)
 				)
@@
 		(in_pos_files yes)
 		(dnp no)
-		(property "Reference" "C5"
+		(property "Reference" "C6"
 			(at 162.56 87.63 90)
 			(show_name no)
@@
 			(project "OBC"
 				(path "/100d4475-6c5b-4ca4-82f4-ff20798e9edf/dc03155b-7cbf-4ee4-9f4c-dba3ed8dc3dd/e4d2ab53-3ce3-4165-a625-695d4175e2ed"
-					(reference "C5")
+					(reference "C6")
 					(unit 1)
 				)
@@
 		(in_pos_files yes)
 		(dnp no)
-		(property "Reference" "C16"
+		(property "Reference" "C17"
 			(at 215.9 50.8 90)
 			(show_name no)
@@
 			(project "OBC"
 				(path "/100d4475-6c5b-4ca4-82f4-ff20798e9edf/dc03155b-7cbf-4ee4-9f4c-dba3ed8dc3dd/e4d2ab53-3ce3-4165-a625-695d4175e2ed"
-					(reference "C16")
+					(reference "C17")
 					(unit 1)
 				)
@@
 		(in_pos_files yes)
 		(dnp no)
-		(property "Reference" "C10"
+		(property "Reference" "C11"
 			(at 193.04 50.8 90)
 			(show_name no)
@@
 			(project "OBC"
 				(path "/100d4475-6c5b-4ca4-82f4-ff20798e9edf/dc03155b-7cbf-4ee4-9f4c-dba3ed8dc3dd/e4d2ab53-3ce3-4165-a625-695d4175e2ed"
-					(reference "C10")
+					(reference "C11")
 					(unit 1)
 				)
@@
 		(in_pos_files yes)
 		(dnp no)
-		(property "Reference" "C2"
+		(property "Reference" "C3"
 			(at 112.522 96.774 0)
 			(show_name no)
@@
 			(project "OBC"
 				(path "/100d4475-6c5b-4ca4-82f4-ff20798e9edf/dc03155b-7cbf-4ee4-9f4c-dba3ed8dc3dd/e4d2ab53-3ce3-4165-a625-695d4175e2ed"
-					(reference "C2")
+					(reference "C3")
 					(unit 1)
 				)
@@
 		(in_pos_files yes)
 		(dnp no)
-		(property "Reference" "C11"
+		(property "Reference" "C12"
 			(at 196.85 50.8 90)
 			(show_name no)
@@
 			(project "OBC"
 				(path "/100d4475-6c5b-4ca4-82f4-ff20798e9edf/dc03155b-7cbf-4ee4-9f4c-dba3ed8dc3dd/e4d2ab53-3ce3-4165-a625-695d4175e2ed"
-					(reference "C11")
+					(reference "C12")
 					(unit 1)
 				)
@@
 		(in_pos_files yes)
 		(dnp no)
-		(property "Reference" "C7"
+		(property "Reference" "C8"
 			(at 181.61 50.8 90)
 			(show_name no)
@@
 			(project "OBC"
 				(path "/100d4475-6c5b-4ca4-82f4-ff20798e9edf/dc03155b-7cbf-4ee4-9f4c-dba3ed8dc3dd/e4d2ab53-3ce3-4165-a625-695d4175e2ed"
-					(reference "C7")
+					(reference "C8")
 					(unit 1)
 				)
@@
 		(in_pos_files yes)
 		(dnp no)
-		(property "Reference" "C19"
+		(property "Reference" "C18"
 			(at 219.71 50.8 90)
 			(show_name no)
@@
 			(project "OBC"
 				(path "/100d4475-6c5b-4ca4-82f4-ff20798e9edf/dc03155b-7cbf-4ee4-9f4c-dba3ed8dc3dd/e4d2ab53-3ce3-4165-a625-695d4175e2ed"
-					(reference "C19")
+					(reference "C18")
 					(unit 1)
 				)
@@
 		(in_pos_files yes)
 		(dnp no)
-		(property "Reference" "C21"
+		(property "Reference" "C20"
 			(at 227.33 50.8 90)
 			(show_name no)
@@
 			(project "OBC"
 				(path "/100d4475-6c5b-4ca4-82f4-ff20798e9edf/dc03155b-7cbf-4ee4-9f4c-dba3ed8dc3dd/e4d2ab53-3ce3-4165-a625-695d4175e2ed"
-					(reference "C21")
+					(reference "C20")
 					(unit 1)
 				)
@@
 		(dnp no)
 		(fields_autoplaced yes)
-		(property "Reference" "#PWR07"
+		(property "Reference" "#PWR022"
 			(at 237.49 38.1 0)
 			(hide yes)
@@
 			(project "OBC"
 				(path "/100d4475-6c5b-4ca4-82f4-ff20798e9edf/dc03155b-7cbf-4ee4-9f4c-dba3ed8dc3dd/e4d2ab53-3ce3-4165-a625-695d4175e2ed"
-					(reference "#PWR07")
+					(reference "#PWR022")
 					(unit 1)
 				)
@@
 		(dnp no)
 		(fields_autoplaced yes)
-		(property "Reference" "#PWR01"
+		(property "Reference" "#PWR018"
 			(at 116.84 105.41 0)
 			(hide yes)
@@
 			(project "OBC"
 				(path "/100d4475-6c5b-4ca4-82f4-ff20798e9edf/dc03155b-7cbf-4ee4-9f4c-dba3ed8dc3dd/e4d2ab53-3ce3-4165-a625-695d4175e2ed"
-					(reference "#PWR01")
+					(reference "#PWR018")
 					(unit 1)
 				)
@@
 		(dnp no)
 		(fields_autoplaced yes)
-		(property "Reference" "#PWR06"
+		(property "Reference" "#PWR021"
 			(at 181.61 43.18 0)
 			(hide yes)
@@
 			(project "OBC"
 				(path "/100d4475-6c5b-4ca4-82f4-ff20798e9edf/dc03155b-7cbf-4ee4-9f4c-dba3ed8dc3dd/e4d2ab53-3ce3-4165-a625-695d4175e2ed"
-					(reference "#PWR06")
+					(reference "#PWR021")
 					(unit 1)
 				)
@@
 		(in_pos_files yes)
 		(dnp no)
-		(property "Reference" "C8"
+		(property "Reference" "C9"
 			(at 185.42 50.8 90)
 			(show_name no)
@@
 			(project "OBC"
 				(path "/100d4475-6c5b-4ca4-82f4-ff20798e9edf/dc03155b-7cbf-4ee4-9f4c-dba3ed8dc3dd/e4d2ab53-3ce3-4165-a625-695d4175e2ed"
-					(reference "C8")
+					(reference "C9")
 					(unit 1)
 				)
@@
 		(dnp no)
 		(fields_autoplaced yes)
-		(property "Reference" "#PWR02"
+		(property "Reference" "#PWR019"
 			(at 152.4 100.33 0)
 			(hide yes)
@@
 			(project "OBC"
 				(path "/100d4475-6c5b-4ca4-82f4-ff20798e9edf/dc03155b-7cbf-4ee4-9f4c-dba3ed8dc3dd/e4d2ab53-3ce3-4165-a625-695d4175e2ed"
-					(reference "#PWR02")
+					(reference "#PWR019")
 					(unit 1)
 				)
@@
 		(in_pos_files yes)
 		(dnp no)
-		(property "Reference" "C4"
+		(property "Reference" "C5"
 			(at 162.306 83.82 90)
 			(show_name no)
@@
 			(project "OBC"
 				(path "/100d4475-6c5b-4ca4-82f4-ff20798e9edf/dc03155b-7cbf-4ee4-9f4c-dba3ed8dc3dd/e4d2ab53-3ce3-4165-a625-695d4175e2ed"
-					(reference "C4")
-					(unit 1)
-				)
+					(reference "C5")
+					(unit 1)
+				)
