File: SATURN/OBC/STM32H7 MCU.kicad_sch (KiCad schematic)
At the start: 8 parts, among them IC1 STM32H735AGI6

Commit message: usb
Parts:
- renumbered C22 to C18, C24 to C19, C23 to C20, D1 to D2, D2 to D3
Connections:
- net USB_FS_ID: now reaches IC1.E10 (PA10)
- net USB_FS_D+: now reaches IC1.E13 (PA12)
- net USB_FS_D-: now reaches IC1.F13 (PA11)
Changed lines of the file:
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@@
+		)
+	)
+	(global_label "USB_FS_D-"
+		(shape input)
+		(at 154.94 284.48 180)
+		(fields_autoplaced yes)
+		(effects
+			(font
+				(size 1.27 1.27)
+			)
+			(justify right)
+		)
+		(property "Intersheetrefs" "${INTERSHEET_REFS}"
+			(at 141.0691 284.48 0)
+			(effects
+				(font
+					(size 1.27 1.27)
+				)
+				(justify right)
+				(hide yes)
+			)
 		)
 	)
@@
 		)
 	)
+	(global_label "USB_FS_D+"
+		(shape input)
+		(at 154.94 251.46 180)
+		(fields_autoplaced yes)
+		(effects
+			(font
+				(size 1.27 1.27)
+			)
+			(justify right)
+		)
+		(property "Intersheetrefs" "${INTERSHEET_REFS}"
+			(at 141.0691 251.46 0)
+			(effects
+				(font
+					(size 1.27 1.27)
+				)
+				(justify right)
+				(hide yes)
+			)
+		)
+	)
 	(global_label "MCU_VSS"
 		(shape input)
@@
 		(property "Intersheetrefs" "${INTERSHEET_REFS}"
 			(at 143.3067 93.98 0)
+			(effects
+				(font
+					(size 1.27 1.27)
+				)
+				(justify right)
+				(hide yes)
+			)
+		)
+	)
+	(global_label "USB_FS_ID"
+		(shape input)
+		(at 154.94 243.84 180)
+		(fields_autoplaced yes)
+		(effects
+			(font
+				(size 1.27 1.27)
+			)
+			(justify right)
+		)
+		(property "Intersheetrefs" "${INTERSHEET_REFS}"
+			(at 142.0367 243.84 0)
 			(effects
 				(font
@@
 		(on_board yes)
 		(dnp no)
-		(property "Reference" "D1"
+		(property "Reference" "D2"
 			(at 213.868 98.806 0)
 			(effects
@@
 		(dnp no)
 		(fields_autoplaced yes)
-		(property "Reference" "#PWR012"
+		(property "Reference" "#PWR?"
 			(at 217.17 113.03 0)
 			(effects
@@
 				(path "/100d4475-6c5b-4ca4-82f4-ff20798e9edf/dc03155b-7cbf-4ee4-9f4c-dba3ed8dc3dd/22739825-328f-4750-87fc-f1f294c30175"
 					(reference "#PWR012")
+					(unit 1)
+				)
+			)
+			(project "STM_Hardware"
+				(path "/3dc4ada8-4f3f-4815-a67d-6c3de6c033d8/22739825-328f-4750-87fc-f1f294c30175"
+					(reference "#PWR?")
 					(unit 1)
 				)
@@
 		(on_board yes)
 		(dnp no)
-		(property "Reference" "C22"
+		(property "Reference" "C18"
 			(at 147.32 132.334 0)
 			(effects
@@
 		(dnp no)
 		(fields_autoplaced yes)
-		(property "Reference" "#PWR09"
+		(property "Reference" "#PWR0102"
 			(at 214.63 101.6 0)
 			(effects
@@
 		(dnp no)
 		(fields_autoplaced yes)
-		(property "Reference" "#PWR08"
+		(property "Reference" "#PWR03"
 			(at 151.13 229.87 0)
 			(effects
@@
 		(dnp no)
 		(fields_autoplaced yes)
-		(property "Reference" "#PWR010"
+		(property "Reference" "#PWR04"
 			(at 226.06 99.06 0)
 			(effects
@@
 		(dnp no)
 		(fields_autoplaced yes)
-		(property "Reference" "C26"
+		(property "Reference" "C?"
 			(at 231.14 102.0514 0)
 			(effects
@@
 				(path "/100d4475-6c5b-4ca4-82f4-ff20798e9edf/dc03155b-7cbf-4ee4-9f4c-dba3ed8dc3dd/22739825-328f-4750-87fc-f1f294c30175"
 					(reference "C26")
+					(unit 1)
+				)
+			)
+			(project "STM_Hardware"
+				(path "/3dc4ada8-4f3f-4815-a67d-6c3de6c033d8/22739825-328f-4750-87fc-f1f294c30175"
+					(reference "C?")
 					(unit 1)
 				)
@@
 		(dnp no)
 		(fields_autoplaced yes)
-		(property "Reference" "#PWR011"
+		(property "Reference" "#PWR05"
 			(at 226.06 217.17 0)
 			(effects
@@
 		(on_board yes)
 		(dnp no)
-		(property "Reference" "C25"
+		(property "Reference" "C?"
 			(at 219.71 103.632 0)
 			(effects
@@
 				(path "/100d4475-6c5b-4ca4-82f4-ff20798e9edf/dc03155b-7cbf-4ee4-9f4c-dba3ed8dc3dd/22739825-328f-4750-87fc-f1f294c30175"
 					(reference "C25")
+					(unit 1)
+				)
+			)
+			(project "STM_Hardware"
+				(path "/3dc4ada8-4f3f-4815-a67d-6c3de6c033d8/22739825-328f-4750-87fc-f1f294c30175"
+					(reference "C?")
 					(unit 1)
 				)
@@
 		(dnp no)
 		(fields_autoplaced yes)
-		(property "Reference" "#PWR013"
+		(property "Reference" "#PWR?"
 			(at 228.6928 112.2052 0)
 			(effects
@@
 				(path "/100d4475-6c5b-4ca4-82f4-ff20798e9edf/dc03155b-7cbf-4ee4-9f4c-dba3ed8dc3dd/22739825-328f-4750-87fc-f1f294c30175"
 					(reference "#PWR013")
+					(unit 1)
+				)
+			)
+			(project "STM_Hardware"
+				(path "/3dc4ada8-4f3f-4815-a67d-6c3de6c033d8/22739825-328f-4750-87fc-f1f294c30175"
+					(reference "#PWR?")
 					(unit 1)
 				)
@@
 		(dnp no)
 		(fields_autoplaced yes)
-		(property "Reference" "C24"
+		(property "Reference" "C19"
 			(at 227.33 205.7399 0)
 			(effects
@@
 		(on_board yes)
 		(dnp no)
-		(property "Reference" "D2"
+		(property "Reference" "D3"
 			(at 220.218 96.266 0)
 			(effects
@@
 		(dnp no)
 		(fields_autoplaced yes)
-		(property "Reference" "C23"
+		(property "Reference" "C20"
 			(at 215.9 207.0162 0)
 			(effects
