File: SATURN/OBC/STM32H7 MCU.kicad_sch (KiCad schematic)
At the start: 8 parts, among them IC1 STM32H735AGI6

Commit message: Wired Up Watchdogs. Hopefully correctly.
Parts:
- renumbered C18 to C22, C20 to C23, C19 to C24, D2 to D1, D3 to D2

Commit message: Update SWD and 3.3V tags
Connections:
- net SWCLK renamed SWDCLK
Changed lines of the file:
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@@
 		)
 	)
-	(global_label "SWCLK"
+	(global_label "SWDCLK"
 		(shape input)
 		(at 154.94 149.86 180)
@@
 		)
 		(property "Intersheetrefs" "${INTERSHEET_REFS}"
-			(at 145.7258 149.86 0)
+			(at 144.4558 149.86 0)
 			(hide yes)
 			(show_name no)

Commit message: Added USB switcher and updated to MCUs
Parts:
- added C26: 10uf, Capacitor_SMD:C_0603_1608Metric, symbol Device:C_Small
- added C27: 100 nF, symbol Device:C_Small
- added C28: 1 uF, symbol Device:C_Small
- added C29: 100 nF, symbol Device:C
- added C30: 4.7 uF, symbol Device:C_Small
- added D3, D4: D_Small, symbol Device:D_Small
- added IC2: STM32H735AGI6, Gabriel_footprints:BGA169C50P13X13_700X700X60, symbol STM32H735AGI6:STM32H735AGI6
- renumbered C22 to C21, C23 to C22, C25 to C23, C26 to C25
Connections:
- net +3.3V: now also C28.1, D3.2 (A)
- net +5V: now also C30.1, D4.2 (A)
- net GND: now also C27.2, C28.2, C29.2, C30.2, IC2.E2 (VSSSMPS), IC2.L4 (PA5)
- net MCU_VDD: now also IC2.A10 (VDD_4), IC2.A3 (VDD_1), IC2.A6 (VDD_2), IC2.A7 (VDD_3), IC2.C13 (VDD_5), IC2.D1 (VDD_6), IC2.G1 (VDD_7), IC2.H13 (VDD_8), IC2.L13 (VDD_9), IC2.M1 (VDD_10), IC2.N11 (VDD_13), IC2.N4 (VDD_11), IC2.N7 (VDD_12)
- net MCU_VDDSMPS: now also IC2.F1 (VDDSMPS)
- net MCU_VFBSMPS: now also C26.2, IC2.B4 (VDDLDO_1), IC2.D12 (VDDLDO_2), IC2.F2 (VFBSMPS), IC2.M10 (VDDLDO_3)
- net MCU_VLXSMPS: now also IC2.E1 (VLXSMPS)
- net MCU_VSS: now also C26.1, IC2.B10 (VSS_3), IC2.B3 (VSS_1), IC2.B7 (VSS_2), IC2.C12 (VSS_4), IC2.D2 (VSS_5), IC2.G2 (VSS_6), IC2.H12 (VSS_7), IC2.L12 (VSS_8), IC2.M11 (VSS_12), IC2.M2 (VSS_9), IC2.M4 (VSS_10), IC2.M7 (VSS_11)
- net SWDCLK: now also IC2.B12 (PA14)
- net SWDIO: now also IC2.D11 (PA13)
- net USB_FS_ID: now also IC2.E10 (PA10)
- net VCAP_1: now also IC2.A4 (VCAP_1)
- net VCAP_2: now also IC2.D13 (VCAP_2)
- net VCAP_3: now also IC2.N10 (VCAP_3)
- net USB_FS_D+ renamed MCU1_USB_FS_D+
- net USB_FS_D- renamed MCU1-USB_FS_D-
- new net: D4.1 (K), IC2.G12 (VDD50USB)
- new net: D3.1 (K), IC2.G13 (VDD33USB)
- new net: C29.1, IC2.L1 (VDDA)
- new net: C27.1, IC2.L2 (VREF+)
- new net MCU1_USB_FS_D-: IC2.F13 (PA11)
- new net MCU2_USB_FS_D+: IC2.E13 (PA12)
Other:
- moved on the sheet: C21, C22, C23, C24, C25, D1, D2, IC1
