File: SATURN/OBC/STM_Hardware.kicad_sch (KiCad schematic)
At the start: 6 parts, among them J1 SWD Pins, P1 USB_C_Plug, U1 STM32H735AGIx

Commit message: Working on STUFF(tm)
Parts:
- removed U1: STM32H735AGIx, Package_BGA:UFBGA-169_7x7mm_Layout13x13_P0.5mm, symbol MCU_ST_STM32H7:STM32H735AGIx
- added C10, C11, C12, C13, C14, C15, C3, C4, C5, C6, C7, C8, C9: 100nf?, symbol Device:C_Small
- added IC1: STM32H735AGI6, BGA169C50P13X13_700X700X60, symbol STM32H735AGI6:STM32H735AGI6
- C1, C2: value C_Small -> 2.2uf
- renumbered D2 to D1
Connections:
- net +3.3V: now also C10.1, C11.1, C12.1, C13.1, C14.1, C15.1, C3.1, C4.1, C5.1, C6.1, C7.1, C8.1, C9.1, IC1.A3 (VDD_1), IC1.A6 (VDD_2), IC1.A7 (VDD_3), IC1.C13 (VDD_5), IC1.D1 (VDD_6), IC1.G1 (VDD_7), IC1.H13 (VDD_8), IC1.L13 (VDD_9), IC1.M1 (VDD_10), IC1.N11 (VDD_13), IC1.N4 (VDD_11), IC1.N7 (VDD_12); no longer C1.2, C2.2
- net at D1.2 (A): now also IC1.G13 (VDD33USB)
- net GND: now reaches C1.1
- net GND: now also C2.1, C10.2, C11.2, C12.2, C13.2, C14.2, C15.2, C3.2, C4.2, C5.2, C6.2, C7.2, C8.2, C9.2, IC1.B10 (VSS_3), IC1.B3 (VSS_1), IC1.B7 (VSS_2), IC1.C12 (VSS_4), IC1.D2 (VSS_5), IC1.G2 (VSS_6), IC1.H12 (VSS_7), IC1.L12 (VSS_8), IC1.M11 (VSS_12), IC1.M2 (VSS_9), IC1.M4 (VSS_10), IC1.M7 (VSS_11)
- new net: C2.2, IC1.D13 (VCAP_2)
- new net: C1.2, IC1.A4 (VCAP_1)
- new net SWCLK: IC1.B12 (PA14)
- new net SWDIO: IC1.D11 (PA13)
Other:
- moved on the sheet: C1, D1, P1

Commit message: wip
Parts:
- removed P1: USB_C_Plug, symbol Connector:USB_C_Plug
- added C16: 4.7uf, Capacitor_SMD:C_0603_1608Metric, symbol Device:C_Small
- added C17: 220pf, Capacitor_SMD:C_0603_1608Metric, symbol Device:C_Small
- added C18, C19: 10uf, Capacitor_SMD:C_0603_1608Metric, symbol Device:C_Small
- added J2: USB_C_Receptacle, symbol Connector:USB_C_Receptacle
- added L1: 2.2uH, symbol Device:L
- C1, C10, C11, C12, C13, C14, C15, C2, C3, C4, C5, C6, C7, C8, C9: footprint (none) -> Capacitor_SMD:C_0603_1608Metric
- IC1: footprint BGA169C50P13X13_700X700X60 -> Gabriel_footprints:BGA169C50P13X13_700X700X60
Connections:
- net +3.3V: now also IC1.A10 (VDD_4), IC1.F1 (VDDSMPS), C16.2
- net GND: now also IC1.E2 (VSSSMPS), C16.1, C17.1, C18.1, C19.1
- net MCU_VFBSMPS: now reaches IC1.B4 (VDDLDO_1)
- net MCU_VFBSMPS: now also IC1.D12 (VDDLDO_2), IC1.F2 (VFBSMPS), IC1.M10 (VDDLDO_3), C18.2, C19.2, L1.2
- net MCU_VLXSMPS: now reaches IC1.E1 (VLXSMPS)
- net MCU_VLXSMPS: now also C17.2, L1.1
- new net: J2.A1 (GND), J2.A12 (GND), J2.B1 (GND), J2.B12 (GND)
- new net: J2.A4 (VBUS), J2.A9 (VBUS), J2.B4 (VBUS), J2.B9 (VBUS)
Other:
- moved on the sheet: C2

Commit message: Messy but working on turing it into a hierarchical schematic
Parts:
- removed C1, C2: 2.2uf, Capacitor_SMD:C_0603_1608Metric, symbol Device:C_Small
- removed C10, C11, C12, C13, C14, C15, C3, C4, C5, C6, C7, C8, C9: 100nf?, Capacitor_SMD:C_0603_1608Metric, symbol Device:C_Small
- removed C16: 4.7uf, Capacitor_SMD:C_0603_1608Metric, symbol Device:C_Small
- removed C19: 10uf, Capacitor_SMD:C_0603_1608Metric, symbol Device:C_Small
- removed D1: D_Small, symbol Device:D_Small
- removed IC1: STM32H735AGI6, Gabriel_footprints:BGA169C50P13X13_700X700X60, symbol STM32H735AGI6:STM32H735AGI6
Other:
- added sheet MCU Power (MCU_Power.kicad_sch)
- added sheet STM32H7 MCU (STM32H7 MCU.kicad_sch)

Commit message: usb
Parts:
- removed J2: USB_C_Receptacle, symbol Connector:USB_C_Receptacle
- added J2: USB_OTG, symbol Connector:USB_OTG
- added U1: USBLC6-4SC6, Package_TO_SOT_SMD:SOT-23-6, symbol Power_Protection:USBLC6-4SC6
Connections:
- net GND: now also J2.5 (GND), J2.6 (Shield), U1.2 (GND)
- new net USB_FS_D+: J2.3 (D+), U1.3 (I/O2)
- new net USB_FS_D-: J2.2 (D-), U1.4 (I/O3)
- new net USB_FS_ID: J2.4 (ID), U1.6 (I/O4)
- no-connect marks 0 -> 1
Other:
- note added: "3.3v tvs diode link, idk if we need a different kind for 3.3 lines"
- note added: "?"
- moved on the sheet: J1
