File: SATURN/OBC/OBC.kicad_pcb (KiCad board)
At the start: 6 copper layers, 16 parts, among them IC1 STM32H735AGI6

Commit message: Buncha changes, had to merge manually, hopefully nothing is broken.
Added the second MCU
Updated USB switcher
Added backup battery to RTC
Parts:
- added C1: 220pf, Capacitor_SMD:C_0603_1608Metric, F.Cu at (163.5, 81.3)
- added C10: 100nf?, Capacitor_SMD:C_0603_1608Metric, F.Cu at (153.5, 81.3)
- added C11: 100nf?, Capacitor_SMD:C_0603_1608Metric, F.Cu at (153.5, 83.8)
- added C12: 100nf?, Capacitor_SMD:C_0603_1608Metric, F.Cu at (153.5, 86.3)
- added C13: 100nf?, Capacitor_SMD:C_0603_1608Metric, F.Cu at (153.5, 88.8)
- added C14: 100nf?, Capacitor_SMD:C_0603_1608Metric, F.Cu at (153.5, 91.3)
- added C15: 100nf?, Capacitor_SMD:C_0603_1608Metric, F.Cu at (153.5, 93.8)
- added C16: 100nf?, Capacitor_SMD:C_0603_1608Metric, F.Cu at (153.5, 96.3)
- added C17: 100nf?, Capacitor_SMD:C_0603_1608Metric, F.Cu at (157.5, 81.3)
- added C18: 100nf?, Capacitor_SMD:C_0603_1608Metric, F.Cu at (157.5, 83.8)
- added C19: 100nf?, Capacitor_SMD:C_0603_1608Metric, F.Cu at (157.5, 86.3)
- added C2: 10uf, Capacitor_SMD:C_0603_1608Metric, F.Cu at (163.5, 83.8)
- added C20: 100nf?, Capacitor_SMD:C_0603_1608Metric, F.Cu at (157.5, 88.8)
- added C21: 10uf, Capacitor_SMD:C_0603_1608Metric, F.Cu at (163.5, 88.3)
- added C26: 10uf, Capacitor_SMD:C_0603_1608Metric, F.Cu at (163.5, 90.8)
- added C3: 4.7uf, Capacitor_SMD:C_0603_1608Metric, F.Cu at (149.5, 81.3)
- added C4: 4.7 uF, Capacitor_SMD:C_0603_1608Metric, F.Cu at (149.5, 83.8)
- added C5: 4.7 uF, Capacitor_SMD:C_0603_1608Metric, F.Cu at (149.5, 86.3)
- added C6: 2.2 uF, Capacitor_SMD:C_0603_1608Metric, F.Cu at (149.5, 88.8)
- added C7: 2.2 uF, Capacitor_SMD:C_0603_1608Metric, F.Cu at (149.5, 91.3)
- added C8: 100nf?, Capacitor_SMD:C_0603_1608Metric, F.Cu at (149.5, 93.8)
- added C9: 100nf?, Capacitor_SMD:C_0603_1608Metric, F.Cu at (149.5, 96.3)
- added J1: SWD Pins, Connector_PinHeader_1.27mm:PinHeader_1x03_P1.27mm_Vertical, F.Cu at (153.1, 65.2)
- added U3: USBLC6-4SC6, Package_TO_SOT_SMD:SOT-23-6, F.Cu at (168.1, 82.4)
- C5: value 100nf? -> 4.7 uF
- C6: value 100nf? -> 2.2 uF
Connections:
- C5 pad 1: MCU_VDD -> MCU_VSS
- C6 pad 1: MCU_VDD -> MCU_VSS
- IC1 pad A10: unconnected-(IC1-VDD_4-PadA10) -> MCU_VDD
- IC1 pad A4: Net-(IC1-VCAP_1) -> MCU_VSS
- IC1 pad B12: SWCLK -> SWDCLK
- IC1 pad B4: unconnected-(IC1-VDDLDO_1-PadB4) -> MCU_VFBSMPS
- IC1 pad D12: unconnected-(IC1-VDDLDO_2-PadD12) -> MCU_VFBSMPS
- IC1 pad D13: Net-(IC1-VCAP_2) -> VCAP_2
- IC1 pad E1: unconnected-(IC1-VLXSMPS-PadE1) -> MCU_VLXSMPS
- IC1 pad E10: unconnected-(IC1-PA10-PadE10) -> USB_FS_ID
- IC1 pad E13: unconnected-(IC1-PA12-PadE13) -> MCU1_USB_FS_D+
- IC1 pad E2: unconnected-(IC1-VSSSMPS-PadE2) -> MCU_VSS
- IC1 pad F1: unconnected-(IC1-VDDSMPS-PadF1) -> MCU_VDD
- IC1 pad F13: unconnected-(IC1-PA11-PadF13) -> MCU1-USB_FS_D-
- IC1 pad F2: unconnected-(IC1-VFBSMPS-PadF2) -> MCU_VFBSMPS
- IC1 pad G12: unconnected-(IC1-VDD50USB-PadG12) -> Net-(D2-K)
- IC1 pad L1: unconnected-(IC1-VDDA-PadL1) -> Net-(IC1-VDDA)
- IC1 pad L2: unconnected-(IC1-VREF+-PadL2) -> Net-(IC1-VREF+)
- IC1 pad L4: unconnected-(IC1-PA5-PadL4) -> MCU_VSS
- IC1 pad M10: unconnected-(IC1-VDDLDO_3-PadM10) -> MCU_VFBSMPS
- IC1 pad N10: unconnected-(IC1-VCAP_3-PadN10) -> MCU_VSS
