File: SATURN/OBC/_restore_backup_2026-08-31T21-15-11-103/MCU_Power.kicad_sch (KiCad schematic)
At the start: 23 parts

Commit message: Buncha changes, had to merge manually, hopefully nothing is broken.
Added the second MCU
Updated USB switcher
Added backup battery to RTC
Parts:
- renumbered C29 to C1, C40 to C10, C41 to C11, C42 to C12, C43 to C13, C44 to C14, C45 to C15, C46 to C16, C32 to C17, C31 to C18, C47 to C19, C30 to C2, C48 to C20, C49 to C21, C33 to C3, C34 to C4, C35 to C5, C36 to C6, C37 to C7, C38 to C8, C39 to C9, L5 to L1, L4 to L2
