File: SATURN/CDH/MCU_Power.kicad_sch (KiCad schematic)
At the start: 23 parts

Commit message: Added memory, connections to MCUs
Parts:
- added C61, C62: 4.7 uF, Capacitor_SMD:C_0603_1608Metric, symbol Device:C_Small
- added C63, C64: 2.2 uF, Capacitor_SMD:C_0603_1608Metric, symbol Device:C_Small
- added C65, C66, C67, C68, C69, C70, C71, C72, C73, C74, C75, C76, C77: 100nf?, Capacitor_SMD:C_0603_1608Metric, symbol Device:C_Small
Connections:
- net +3.3V: now also C65.1, C66.1, C67.1, C68.1, C69.1, C70.1, C71.1, C72.1, C73.1, C74.1, C75.1, C76.1, C77.1
- net GND: now also C61.1, C61.2, C62.1, C62.2, C63.1, C63.2, C64.2, C65.2, C66.2, C67.2, C68.2, C69.2, C70.2, C71.2, C72.2, C73.2, C74.2, C75.2, C76.2, C77.2
- net VCAP_2 renamed VCAP_2A
- new net VCAP_2B: C64.1
Other:
- moved on the sheet: C37, C38, C39, C40, C41, C42, C43, C44, C45, C46, C47, C48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
