File: SATURN/CDH/STM32H7 MCU.kicad_sch (KiCad schematic)
At the start: 24 parts, among them IC1 STM32H735AGI6, IC2 STM32H735AGI6, IC3 STM32H735AGI6

Commit message: Added memory, connections to MCUs
Parts:
- removed C18, C26: 10uf, Capacitor_SMD:C_0603_1608Metric, symbol Device:C_Small
- removed C19, C52: 100 nF, symbol Device:C
- removed C20, C50: 100 nF, symbol Device:C_Small
- removed C21, C51: 1 uF, symbol Device:C_Small
- removed C22, C53: 4.7 uF, symbol Device:C_Small
- removed D2, D3, D4, D5: D_Small, symbol Device:D_Small
- removed IC3: STM32H735AGI6, Gabriel_footprints:BGA169C50P13X13_700X700X60, symbol STM32H735AGI6:STM32H735AGI6
- added C56: 10uf, Capacitor_SMD:C_0603_1608Metric, symbol Device:C_Small
- added C57: 100 nF, symbol Device:C_Small
- added C58: 100 nF, symbol Device:C
- added C59: 1 uF, symbol Device:C_Small
- added C60: 4.7 uF, symbol Device:C_Small
- added D7, D8: D_Small, symbol Device:D_Small
Connections:
- net MCU1-USB_FS_D- is gone; now on net USB_FS_D-: IC1.F13 (PA11)
- net MCU1_USB_FS_D+ is gone; now on net USB_FS_D+: IC1.E13 (PA12)
- net MCU1_USB_FS_D- is gone; now on net USB_FS_D-: IC2.F13 (PA11)
- net MCU2_USB_FS_D+ is gone; now on net USB_FS_D+: IC2.E13 (PA12)
- net +3.3V: now also C59.1, D7.2 (A)
- net +5V: now also C60.1, D8.2 (A)
- net FDCAN1_RX: now also IC1.A13 (PH14), IC2.A13 (PH14)
- net FDCAN1_TX: now also IC1.B13 (PH13), IC2.B13 (PH13)
- net FMC_ALE: now also IC1.K13 (PD12), IC2.K13 (PD12)
- net FMC_CLE: now also IC1.J10 (PD11), IC2.J10 (PD11)
- net FMC_D0: now also IC1.J13 (PD14), IC2.J13 (PD14)
- net FMC_D1: now also IC1.J12 (PD15), IC2.J12 (PD15)
- net FMC_D2: now also IC1.D10 (PD0), IC2.D10 (PD0)
- net FMC_D3: now also IC1.C10 (PD1), IC2.C10 (PD1)
- net FMC_D4: now also IC1.G8 (PE7), IC2.G8 (PE7)
- net FMC_D5: now also IC1.H8 (PE8), IC2.H8 (PE8)
- net FMC_D6: now also IC1.A11 (PC12), IC2.A11 (PC12)
- net FMC_D7: now also IC1.E9 (PD2), IC2.E9 (PD2)
- net FMC_NOE: now also IC1.C9 (PD4), IC2.C9 (PD4)
- net FMC_NWE: now also IC1.A9 (PD5), IC2.A9 (PD5)
- net GND: now also C57.2, C58.2, C59.2, C60.2
- net I2C1_SDA: now also IC1.C5 (PB9), IC2.C5 (PB9)
- net I2C2_SCL: now also IC1.E4 (PF1), IC2.E4 (PF1)
- net I2C2_SDA: now also IC1.F3 (PF0), IC2.F3 (PF0)
- net MCU_VDD: now also IC1.E3 (VBAT), IC2.E3 (VBAT)
- net MCU_VFBSMPS: now also C56.2
- net MCU_VSS: now also C56.1
- net OCTOSPIM_P1_CLK: now also IC1.H3 (PF10), IC2.H3 (PF10)
- net OCTOSPIM_P1_IO0: now also IC1.F11 (PC9), IC2.F11 (PC9)
- net OCTOSPIM_P1_IO1: now also IC1.A12 (PC10), IC2.A12 (PC10)
- net OCTOSPIM_P1_IO2: now also IC1.A2 (PE2), IC2.A2 (PE2)
- net OCTOSPIM_P1_IO3: now also IC1.G4 (PF6), IC2.G4 (PF6)
- net OCTOSPIM_P1_NCS: now also IC1.B11 (PC11), IC2.B11 (PC11)
- net RCC_OSC32_IN: now also IC1.C1 (PC14-_OSC32_IN), IC2.C1 (PC14-_OSC32_IN)
- net RCC_OSC32_OUT: now also IC1.B1 (PC15-_OSC32_OUT), IC2.B1 (PC15-_OSC32_OUT)
- net RCC_OSC_IN: now also IC1.H1 (PH0-OSC_IN), IC2.H1 (PH0-OSC_IN)
- net RCC_OSC_OUT: now also IC1.H2 (PH1-_OSC_OUT), IC2.H2 (PH1-_OSC_OUT)
- net SPI1_MISO: now also IC1.B6 (PB4), IC2.B6 (PB4)
- net SPI1_MOSI: now also IC1.C6 (PB5), IC2.C6 (PB5)
- net SPI1_SCK: now also IC1.B8 (PG11), IC2.B8 (PG11)
- net UART4_RX: now also IC1.B5 (PB8), IC2.B5 (PB8)
- net UART4_TX: now also IC1.J5 (PA0), IC2.J5 (PA0)
- net USB_FS_ID: now also IC1.E10 (PA10), IC2.E10 (PA10)
- net USB_FS_VBUS: now also IC1.E11 (PA9), IC2.E11 (PA9)
- net at IC2.G12 (VDD50USB): now also D6.1 (K)
- net at IC2.G13 (VDD33USB): now also D1.1 (K)
- net at C25.1: now also IC2.L1 (VDDA)
- net MCU_RESET: now reaches IC2.G6 (NRST)
- net MCU_RESET: now also IC1.G6 (NRST)
- net FDCAN2_TX: now reaches IC2.L11 (PB13)
- net FDCAN2_TX: now also IC1.L11 (PB13)
- net at IC2.L2 (VREF+): now also C24.1
- net FDCAN2_RX: now reaches IC2.N12 (PB12)
- net FDCAN2_RX: now also IC1.N12 (PB12)
- net at IC1.G12 (VDD50USB): now also D8.1 (K)
- net at IC1.G13 (VDD33USB): now also D7.1 (K)
- net FMC_NWAIT: now reaches IC1.B9 (PD6)
- net FMC_NCE: now reaches IC1.C8 (PG9)
- net at IC1.L1 (VDDA): now also C58.1
- net at IC1.L2 (VREF+): now also C57.1
- net VCAP_1 renamed VCAP_1A
- net VCAP_1A: no longer IC2.A4 (VCAP_1)
- net VCAP_2 renamed VCAP_2A
- net VCAP_2A: no longer IC2.D13 (VCAP_2)
- net VCAP_3 renamed VCAP_3A
- net VCAP_3A: no longer IC2.N10 (VCAP_3)
- new net VCAP_1B: IC2.A4 (VCAP_1)
- new net VCAP_2B: IC2.D13 (VCAP_2)
- new net VCAP_3B: IC2.N10 (VCAP_3)
Other:
- moved on the sheet: C23, C24, C25, C54, C55, D1, D6
