File: SATURN/EPS/EPS/EPS.kicad_sch (KiCad schematic)
At the start: 24 parts, among them IC1 BQ25792RQMR, IC2 BQ25792RQMR, J1 Conn_01x02_Pin, U1 TPS2121RUXR, U2 TPS2121RUXR, U3 MAX25239AFFD/VY+

Commit message: There are in fact some changes
I put a few symbols on there and then hooked up a bunch of them. I *feel* like I'm doing something wrong because this is so confusing, but there is some work there at least
Parts:
- removed IC2: BQ25792RQMR, BQ25792RQMR, symbol SATURN:BQ25792RQMR
- added C1: 1-µF, symbol Device:C_Small
- added C10, C11: 4.7μF, symbol Device:C_Small
- added C2: 0.47μF, symbol Device:C_Small
- added C3: 0.1μF, symbol Device:C_Small
- added Q1, Q2: AON6276, DFN5X6_8L_EP1_P_AOS, symbol SATURN:AON6276
- added R11, R8, R9: 10kΩ, symbol Device:R_Small_US
- added R4: 2mΩ, symbol Device:R_Small_US
- added R5, R6, R7: TBD, symbol Device:R_Small_US
- added TH2: 10-kΩ, symbol Device:Thermistor_US
- added U4: BQ25820RRVR, BQ25820RRVR:IC_BQ25820RRVR, symbol SATURN:BQ25820RRVR
Connections:
- net +3V3: now also R11.2
- net GND: now also C1.2, R9.1
- net MUXOUT: now also C1.1, Q1.5, Q1.6, Q1.7, Q1.8, U4.33 (VAC)
- new net: R5.2, R6.2, TH2.1
- new net: TH2.2, U4.8 (TS)
- new net: R7.1, U4.11 (FBG)
- new net: C2.2, C3.1, U4.13 (SRN)
- new net: C2.1, U4.14 (SRP)
- new net: C10.1, U4.23 (DRV_SUP)
- new net: C11.2, U4.24 (REGN)
- new net: R8.1, U4.3 (~{INT})
- new net: R9.2, U4.7 (~{CE})
- new net ACDRV: U4.31 (ACDRV)
- new net ACN: R4.2, U4.29 (ACN), U4.32 (SYS)
- new net ACP: Q2.5, Q2.6, Q2.7, Q2.8, R4.1, U4.30 (ACP)
- new net BATDRV: Q1.4, Q2.4, U4.16 (BATSRC)
- new net BATSRC: Q1.1, Q1.2, Q1.3, Q2.1, Q2.2, Q2.3
- new net EPSSCL: U4.1 (SCL)
- new net EPSSDA: U4.2 (SDA)
- new net PGND: C10.2, C11.1, C3.2, R6.1, U4.10 (ILIM_HIZ), U4.22 (PGND), U4.37 (PGND__1), U4.9 (ICHG)
- new net PWR_GOOD: R11.1, U4.4 (STAT1), U4.5 (STAT2), U4.6 (~{PG})
- new net PWR_INT: R8.2
- new net REGN: R5.1
Other:
- note added: "Battery Feedback Resistor"
- note added: "Battery Temp Thermistor"
- note added: "I pinned Charge Enable to a pull down so that it is always charging, I figure that is fine (if it isn't lmk)"
- note added: "I waited on hooking this up because it is a boost converter and we don't need a boost as we already have 14.4V"
- moved on the sheet: J1, U3
